File: pcb/stm8l-lora-sensor.sch (KiCad schematic (older format))
At the start: 20 parts, among them J1 Conn_01x03, J2 Conn_01x03, J3 Conn_01x02, SW1 SW_Push, U1 BME280, U2 STM8L051F3P, U3 Ai-Thinker-Ra-01, U4 LP2985-3.3, Y1 Crystal

Commit message: sch done, but requires rethink
Parts:
- removed SW1: SW_Push, symbol Switch:SW_Push
- removed U1: BME280, Package_LGA:LGA-8_2.5x2.5mm_P0.65mm, symbol Sensor:BME280
- removed U?: 74HC595, symbol Logic_74xx:74HC595
- added J1: Conn_01x06, Connector_PinHeader_2.54mm:PinHeader_1x06_P2.54mm_Vertical, symbol Connector_Generic:Conn_01x06
- added J2, J6: Conn_01x02, Connector_PinHeader_2.54mm:PinHeader_1x02_P2.54mm_Vertical, symbol Connector_Generic:Conn_01x02
- added R1, R10: 10k, Resistor_SMD:R_0805_2012Metric, symbol Device:R
- added R15, R16, R17, R18: 100k, Resistor_SMD:R_0805_2012Metric, symbol Device:R
- added R2, R3, R4, R5, R6, R7, R8, R9: 1k, Resistor_SMD:R_0805_2012Metric, symbol Device:R
- added U4: CA56-12EWA, Display_7Segment:CA56-12EWA, symbol Display_Character:CA56-12EWA
- C1, C2, C3, C4: footprint (none) -> Capacitor_SMD:C_0805_2012Metric
- J3: renamed from J1; footprint (none) -> Connector_PinHeader_2.54mm:PinHeader_1x03_P2.54mm_Vertical
- J4: renamed from J2; footprint (none) -> Connector_PinHeader_2.54mm:PinHeader_1x03_P2.54mm_Vertical
- J5: renamed from J3; footprint (none) -> Connector_PinHeader_2.54mm:PinHeader_1x02_P2.54mm_Vertical
- R11: renamed from R3; footprint (none) -> Resistor_SMD:R_0805_2012Metric
- R12: renamed from R1; footprint (none) -> Resistor_SMD:R_0805_2012Metric
- R13: renamed from R2; footprint (none) -> Resistor_SMD:R_0805_2012Metric
- R14: renamed from R4; footprint (none) -> Resistor_SMD:R_0805_2012Metric
- U1, U3: renamed from U?; footprint (none) -> Package_SO:SOIC-16_3.9x9.9mm_P1.27mm
- Y1: footprint (none) -> Crystal:Crystal_C26-LF_D2.1mm_L6.5mm_Horizontal
- renumbered U3 to U5, U4 to U6
Connections:
- wire segments 85 -> 143
- no-connect marks 9 -> 14

Commit message: sensor back on i2c
Parts:
- added R19, R20: 10k, Resistor_SMD:R_0805_2012Metric, symbol Device:R
Connections:
- net labels added: SCL, SDA
- net labels removed: CS_SENSOR
- wire segments 143 -> 154
- no-connect marks 14 -> 13
Other:
- note added: "BME280 Sensor:\nCSB to VSS = I2C interface\nSDO to GND = Default Address"
Changed lines of the file:
@@
 Wire Wire Line
 	9250 1000 9350 1000
-Text GLabel 9250 1400 0    50   Output ~ 0
+Text GLabel 9250 1400 0    50   BiDi ~ 0
 SWIM
-Text GLabel 8750 1500 0    50   Input ~ 0
+Text GLabel 8750 1500 0    50   Output ~ 0
 RST
 Wire Wire Line
@@
 Wire Wire Line
 	8750 1500 8850 1500
-Text GLabel 3600 1450 0    50   Input ~ 0
+Text GLabel 3600 1450 0    50   BiDi ~ 0
 SWIM
 Text GLabel 3600 1550 0    50   Input ~ 0
@@
 Wire Wire Line
 	3600 2650 3700 2650
-NoConn ~ 3700 2350
-Text GLabel 5000 1450 2    50   Output ~ 0
+Text GLabel 3600 2350 0    50   Output ~ 0
 CS_LORA
-Text GLabel 5000 1550 2    50   Output ~ 0
-CS_SENSOR
 Text GLabel 5000 1650 2    50   Input ~ 0
 BTN
 Wire Wire Line
-	4900 1450 5000 1450
-Wire Wire Line
-	4900 1550 5000 1550
+	4900 1450 5200 1450
+Wire Wire Line
+	4900 1550 4950 1550
 Wire Wire Line
 	4900 1650 5000 1650
@@
 Wire Wire Line
 	5100 1850 4900 1850
-Text GLabel 1450 1900 2    50   Output ~ 0
-SPI1_MISO
 Text GLabel 1450 1600 2    50   Input ~ 0
-SPI1_SCK
-Text GLabel 1450 1700 2    50   Input ~ 0
-SPI1_MOSI
-Text GLabel 1450 1800 2    50   Input ~ 0
-CS_SENSOR
+SCL
+Text GLabel 1450 1700 2    50   BiDi ~ 0
+SDA
 NoConn ~ 7000 1400
 Text GLabel 6900 1800 0    50   Input ~ 0
@@
 Wire Wire Line
 	9950 3100 10100 3100
-Text GLabel 7550 4550 0    50   Input ~ 0
+Text GLabel 7550 4550 0    50   Output ~ 0
 BTN
 $Comp
@@
 	1350 1700 1450 1700
 Wire Wire Line
-	1350 1800 1450 1800
-Wire Wire Line
 	1350 1900 1450 1900
 $Comp
@@
 	7550 4550 7700 4550
 Connection ~ 7700 4550
+Wire Wire Line
+	3700 2350 3600 2350
+Text GLabel 5300 1550 2    50   Output ~ 0
+SCL
+Text GLabel 5300 1450 2    50   BiDi ~ 0
+SDA
+$Comp
+L Device:R R19
+U 1 1 5AEDD233
+P 4950 1200
+F 0 "R19" H 4880 1154 50  0000 R CNN
+F 1 "10k" H 4880 1245 50  0000 R CNN
+F 2 "Resistor_SMD:R_0805_2012Metric" V 4880 1200 50  0001 C CNN
+F 3 "~" H 4950 1200 50  0001 C CNN
+	1    4950 1200
+	-1   0    0    1
+$EndComp
+$Comp
+L Device:R R20
+U 1 1 5AEDD2C1
+P 5200 1200
+F 0 "R20" H 5130 1154 50  0000 R CNN
+F 1 "10k" H 5130 1245 50  0000 R CNN
+F 2 "Resistor_SMD:R_0805_2012Metric" V 5130 1200 50  0001 C CNN
+F 3 "~" H 5200 1200 50  0001 C CNN
+	1    5200 1200
+	-1   0    0    1
+$EndComp
+Wire Wire Line
+	4950 1350 4950 1550
+Connection ~ 4950 1550
+Wire Wire Line
+	4950 1550 5300 1550
+Wire Wire Line
+	5200 1350 5200 1450
+Connection ~ 5200 1450
+Wire Wire Line
+	5200 1450 5300 1450
+Wire Wire Line
+	4950 1050 4950 1000
+Wire Wire Line
+	4950 1000 5050 1000
+Wire Wire Line
+	5200 1000 5200 1050
+$Comp
+L power:VCC #PWR0101
+U 1 1 5AEF267E
+P 5050 1000
+F 0 "#PWR0101" H 5050 850 50  0001 C CNN
+F 1 "VCC" H 5067 1173 50  0000 C CNN
+F 2 "" H 5050 1000 50  0001 C CNN
+F 3 "" H 5050 1000 50  0001 C CNN
+	1    5050 1000
+	1    0    0    -1
+$EndComp
+Connection ~ 5050 1000
+Wire Wire Line
+	5050 1000 5200 1000
+Wire Wire Line
+	2050 1400 2300 1400
+Connection ~ 2050 1400
+Wire Wire Line
+	1350 1800 2300 1800
+Wire Wire Line
+	2300 1400 2300 1800
+$Comp
+L power:GND #PWR0102
+U 1 1 5AF2B9FF
+P 1450 1900
+F 0 "#PWR0102" H 1450 1650 50  0001 C CNN
+F 1 "GND" H 1455 1727 50  0000 C CNN
+F 2 "" H 1450 1900 50  0001 C CNN
+F 3 "" H 1450 1900 50  0001 C CNN
+	1    1450 1900
+	1    0    0    -1
+$EndComp
+Text Notes 1100 2400 0    50   ~ 0
+BME280 Sensor:\nCSB to VSS = I2C interface\nSDO to GND = Default Address
 $EndSCHEMATC

Commit message: pcb placement done. Have to change LED indicator
Parts:
- removed J4: Conn_01x03, Connector_PinHeader_2.54mm:PinHeader_1x03_P2.54mm_Vertical, symbol Connector_Generic:Conn_01x03
- added C2, C5: 4.7u, Capacitor_SMD:C_0805_2012Metric, symbol Device:C
- added D1: LED, LED_SMD:LED_0805_2012Metric, symbol Device:LED
- added J3: Conn_01x04, Connector_PinHeader_2.54mm:PinHeader_1x04_P2.54mm_Vertical, symbol Connector_Generic:Conn_01x04
- added R20: 2k, Resistor_SMD:R_0805_2012Metric, symbol Device:R
- added R22: 470, Resistor_SMD:R_0805_2012Metric, symbol Device:R
- added U6: MCP73831-2-OT, Package_TO_SOT_SMD:SOT-23-5, symbol Battery_Management:MCP73831-2-OT
- renumbered C2 to C4, C4 to C6, J3 to J4, R15 to R1, R6 to R10, R7 to R11, R8 to R12, R9 to R13, R10 to R14, R19 to R15, R20 to R16, R12 to R17, R13 to R18, R11 to R19, R16 to R2, R14 to R21, R1 to R3, R17 to R4, R18 to R5, R2 to R6, R3 to R7, R4 to R8, R5 to R9, U6 to U7
Connections:
- net labels added: +BATT
- wire segments 154 -> 182
Other:
- note added: "Actual PN: LP5907MFX-3.3/NOPB"
- note added: "Battery"
- note added: "Button"
- note added: "Debug"
- note added: "Programming"
- note added: "Ratio 1:1\n4.2V -> 2.1V"
- note added: "Ratio 1:1\n6V->3V"
- note added: "Solar, 7V MAX!"
- moved on the sheet: U7

Commit message: pwr flags added
Parts:
- R20: value 2k -> 10k
Connections:
- wire segments 182 -> 184
Changed lines of the file:
@@
 L power:+5V #PWR030
 U 1 1 5AB582DA
-P 10200 1550
-F 0 "#PWR030" H 10200 1400 50  0001 C CNN
-F 1 "+5V" H 10215 1723 50  0000 C CNN
-F 2 "" H 10200 1550 50  0001 C CNN
-F 3 "" H 10200 1550 50  0001 C CNN
-	1    10200 1550
+P 9900 1700
+F 0 "#PWR030" H 9900 1550 50  0001 C CNN
+F 1 "+5V" H 9915 1873 50  0000 C CNN
+F 2 "" H 9900 1700 50  0001 C CNN
+F 3 "" H 9900 1700 50  0001 C CNN
+	1    9900 1700
 	1    0    0    -1
 $EndComp
@@
 L Connector_Generic:Conn_01x02 J5
 U 1 1 5AB585A3
-P 10500 1550
-F 0 "J5" H 10580 1542 50  0000 L CNN
-F 1 "Conn_01x02" H 10580 1451 50  0000 L CNN
-F 2 "Connector_PinHeader_2.54mm:PinHeader_1x02_P2.54mm_Vertical" H 10500 1550 50  0001 C CNN
-F 3 "~" H 10500 1550 50  0001 C CNN
-	1    10500 1550
+P 10550 1700
+F 0 "J5" H 10630 1692 50  0000 L CNN
+F 1 "Conn_01x02" H 10630 1601 50  0000 L CNN
+F 2 "Connector_PinHeader_2.54mm:PinHeader_1x02_P2.54mm_Vertical" H 10550 1700 50  0001 C CNN
+F 3 "~" H 10550 1700 50  0001 C CNN
+	1    10550 1700
 	1    0    0    -1
 $EndComp
@@
 L power:GND #PWR031
 U 1 1 5AB5A39D
-P 10200 1650
-F 0 "#PWR031" H 10200 1400 50  0001 C CNN
-F 1 "GND" H 10205 1477 50  0000 C CNN
-F 2 "" H 10200 1650 50  0001 C CNN
-F 3 "" H 10200 1650 50  0001 C CNN
-	1    10200 1650
-	1    0    0    -1
-$EndComp
-Wire Wire Line
-	10300 1550 10200 1550
-Wire Wire Line
-	10200 1650 10300 1650
+P 9900 1800
+F 0 "#PWR031" H 9900 1550 50  0001 C CNN
+F 1 "GND" H 9905 1627 50  0000 C CNN
+F 2 "" H 9900 1800 50  0001 C CNN
+F 3 "" H 9900 1800 50  0001 C CNN
+	1    9900 1800
+	1    0    0    -1
+$EndComp
+Wire Wire Line
+	10350 1700 10250 1700
+Wire Wire Line
+	9900 1800 10250 1800
 $Comp
 L Regulator_Linear:LP2985-3.3 U7
@@
 P 8500 4550
 F 0 "R20" H 8430 4504 50  0000 R CNN
-F 1 "2k" H 8430 4595 50  0000 R CNN
+F 1 "10k" H 8430 4595 50  0000 R CNN
 F 2 "Resistor_SMD:R_0805_2012Metric" V 8430 4550 50  0001 C CNN
 F 3 "~" H 8500 4550 50  0001 C CNN
@@
 Text Notes 10600 3950 0    50   ~ 0
 Battery
-Text Notes 10450 1450 0    50   ~ 0
+Text Notes 10500 1600 0    50   ~ 0
 Solar, 7V MAX!
 Text Notes 10450 650  0    50   ~ 0
@@
 Wire Wire Line
 	1450 1900 1450 1950
+$Comp
+L power:PWR_FLAG #FLG?
+U 1 1 5ADBE069
+P 10250 1700
+F 0 "#FLG?" H 10250 1775 50  0001 C CNN
+F 1 "PWR_FLAG" H 10250 1874 50  0000 C CNN
+F 2 "" H 10250 1700 50  0001 C CNN
+F 3 "" H 10250 1700 50  0001 C CNN
+	1    10250 1700
+	1    0    0    -1
+$EndComp
+$Comp
+L power:PWR_FLAG #FLG?
+U 1 1 5ADBE10C
+P 10250 1800
+F 0 "#FLG?" H 10250 1875 50  0001 C CNN
+F 1 "PWR_FLAG" H 10250 1973 50  0000 C CNN
+F 2 "" H 10250 1800 50  0001 C CNN
+F 3 "" H 10250 1800 50  0001 C CNN
+	1    10250 1800
+	-1   0    0    1
+$EndComp
+Connection ~ 10250 1800
+Wire Wire Line
+	10250 1800 10350 1800
+Connection ~ 10250 1700
+Wire Wire Line
+	10250 1700 9900 1700
 $EndSCHEMATC

Commit message: Added bypass caps, started pcb
Parts:
- added C10, C11, C7, C8, C9: 0.1u, Capacitor_SMD:C_0805_2012Metric, symbol Device:C
Connections:
- wire segments 184 -> 201
Other:
- note added: "R20 10k=100mA charge current"
Changed lines of the file:
@@
 L power:VCC #PWR06
 U 1 1 5AB26559
-P 2050 1400
-F 0 "#PWR06" H 2050 1250 50  0001 C CNN
-F 1 "VCC" H 2067 1573 50  0000 C CNN
-F 2 "" H 2050 1400 50  0001 C CNN
-F 3 "" H 2050 1400 50  0001 C CNN
-	1    2050 1400
+P 2050 1300
+F 0 "#PWR06" H 2050 1150 50  0001 C CNN
+F 1 "VCC" H 2067 1473 50  0000 C CNN
+F 2 "" H 2050 1300 50  0001 C CNN
+F 3 "" H 2050 1300 50  0001 C CNN
+	1    2050 1300
 	1    0    0    -1
 $EndComp
@@
 $EndComp
 Wire Wire Line
-	4300 1050 4300 1150
-Wire Wire Line
-	7500 1000 7500 1100
+	4300 1050 4300 1100
+Wire Wire Line
+	7500 1000 7500 1050
 $Comp
 L Connector_Generic:Conn_01x03 J4
@@
 $EndComp
 Wire Wire Line
-	2300 3900 2300 4000
+	2300 3900 2300 3950
 $Comp
 L Device:R R3
@@
 $EndComp
 Wire Wire Line
-	4900 5400 4900 5500
+	4900 5400 4900 5450
 $Comp
 L power:GND #PWR014
@@
 L power:GND #PWR07
 U 1 1 5AB267BF
-P 2050 1500
-F 0 "#PWR07" H 2050 1250 50  0001 C CNN
-F 1 "GND" H 2055 1327 50  0000 C CNN
-F 2 "" H 2050 1500 50  0001 C CNN
-F 3 "" H 2050 1500 50  0001 C CNN
-	1    2050 1500
-	1    0    0    -1
-$EndComp
-Wire Wire Line
-	1350 1400 2050 1400
-Wire Wire Line
-	1350 1500 2050 1500
+P 1750 1500
+F 0 "#PWR07" H 1750 1250 50  0001 C CNN
+F 1 "GND" H 1755 1327 50  0000 C CNN
+F 2 "" H 1750 1500 50  0001 C CNN
+F 3 "" H 1750 1500 50  0001 C CNN
+	1    1750 1500
+	1    0    0    -1
+$EndComp
+Wire Wire Line
+	1350 1500 1750 1500
 Wire Wire Line
 	1350 1600 1450 1600
@@
 	5050 1000 5200 1000
 Wire Wire Line
-	2050 1400 2300 1400
-Connection ~ 2050 1400
-Wire Wire Line
-	1350 1800 2300 1800
-Wire Wire Line
-	2300 1400 2300 1800
+	1350 1800 2250 1800
+Wire Wire Line
+	2250 1400 2250 1800
 $Comp
 L power:GND #PWR04
@@
 	1450 1900 1450 1950
 $Comp
-L power:PWR_FLAG #FLG?
+L power:PWR_FLAG #FLG01
 U 1 1 5ADBE069
 P 10250 1700
-F 0 "#FLG?" H 10250 1775 50  0001 C CNN
+F 0 "#FLG01" H 10250 1775 50  0001 C CNN
 F 1 "PWR_FLAG" H 10250 1874 50  0000 C CNN
 F 2 "" H 10250 1700 50  0001 C CNN
@@
 $EndComp
 $Comp
-L power:PWR_FLAG #FLG?
+L power:PWR_FLAG #FLG02
 U 1 1 5ADBE10C
 P 10250 1800
-F 0 "#FLG?" H 10250 1875 50  0001 C CNN
+F 0 "#FLG02" H 10250 1875 50  0001 C CNN
 F 1 "PWR_FLAG" H 10250 1973 50  0000 C CNN
 F 2 "" H 10250 1800 50  0001 C CNN
@@
 Wire Wire Line
 	10250 1700 9900 1700
+Text Notes 9500 5100 2    50   ~ 0
+R20 10k=100mA charge current
+$Comp
+L Device:C C11
+U 1 1 5AE18D04
+P 7750 1050
+F 0 "C11" H 7865 1096 50  0000 L CNN
+F 1 "0.1u" H 7865 1005 50  0000 L CNN
+F 2 "Capacitor_SMD:C_0805_2012Metric" H 7788 900 50  0001 C CNN
+F 3 "~" H 7750 1050 50  0001 C CNN
+	1    7750 1050
+	0    1    1    0
+$EndComp
+$Comp
+L power:GND #PWR037
+U 1 1 5AE18E54
+P 8000 1050
+F 0 "#PWR037" H 8000 800 50  0001 C CNN
+F 1 "GND" H 8005 877 50  0000 C CNN
+F 2 "" H 8000 1050 50  0001 C CNN
+F 3 "" H 8000 1050 50  0001 C CNN
+	1    8000 1050
+	1    0    0    -1
+$EndComp
+Wire Wire Line
+	7500 1050 7600 1050
+Connection ~ 7500 1050
+Wire Wire Line
+	7500 1050 7500 1100
+Wire Wire Line
+	7900 1050 8000 1050
+$Comp
+L power:GND #PWR035
+U 1 1 5AE4D13E
+P 3650 1100
+F 0 "#PWR035" H 3650 850 50  0001 C CNN
+F 1 "GND" H 3655 927 50  0000 C CNN
+F 2 "" H 3650 1100 50  0001 C CNN
+F 3 "" H 3650 1100 50  0001 C CNN
+	1    3650 1100
+	1    0    0    -1
+$EndComp
+$Comp
+L Device:C C9
+U 1 1 5AE4D144
+P 4050 1100
+F 0 "C9" V 3798 1100 50  0000 C CNN
+F 1 "0.1u" V 3889 1100 50  0000 C CNN
+F 2 "Capacitor_SMD:C_0805_2012Metric" H 4088 950 50  0001 C CNN
+F 3 "~" H 4050 1100 50  0001 C CNN
+	1    4050 1100
+	0    1    1    0
+$EndComp
+Wire Wire Line
+	3650 1100 3900 1100
+Wire Wire Line
+	4200 1100 4300 1100
+Connection ~ 4300 1100
+Wire Wire Line
+	4300 1100 4300 1150
+$Comp
+L Device:C C8
+U 1 1 5AE6CF2A
+P 2150 1550
+F 0 "C8" V 1898 1550 50  0000 C CNN
+F 1 "0.1u" V 1989 1550 50  0000 C CNN
+F 2 "Capacitor_SMD:C_0805_2012Metric" H 2188 1400 50  0001 C CNN
+F 3 "~" H 2150 1550 50  0001 C CNN
+	1    2150 1550
+	-1   0    0    1
+$EndComp
+Wire Wire Line
+	1350 1400 2050 1400
+Wire Wire Line
+	2050 1300 2050 1400
+Connection ~ 2050 1400
+Wire Wire Line
+	2050 1400 2150 1400
+Connection ~ 2150 1400
+Wire Wire Line
+	2150 1400 2250 1400
+Wire Wire Line
+	2150 1700 1950 1700
+Wire Wire Line
+	1950 1700 1950 1500
+Wire Wire Line
+	1950 1500 1750 1500
+Connection ~ 1750 1500
+$Comp
+L power:GND #PWR034
+U 1 1 5AEFBFB0
+P 1800 3950
+F 0 "#PWR034" H 1800 3700 50  0001 C CNN
+F 1 "GND" H 1805 3777 50  0000 C CNN
+F 2 "" H 1800 3950 50  0001 C CNN
+F 3 "" H 1800 3950 50  0001 C CNN
+	1    1800 3950
+	1    0    0    -1
+$EndComp
+$Comp
+L Device:C C7
+U 1 1 5AEFBFB6
+P 2050 3950
+F 0 "C7" V 1798 3950 50  0000 C CNN
+F 1 "0.1u" V 1889 3950 50  0000 C CNN
+F 2 "Capacitor_SMD:C_0805_2012Metric" H 2088 3800 50  0001 C CNN
+F 3 "~" H 2050 3950 50  0001 C CNN
+	1    2050 3950
+	0    1    1    0
+$EndComp
+Wire Wire Line
+	1800 3950 1900 3950
+Wire Wire Line
+	2300 3950 2200 3950
+Connection ~ 2300 3950
+Wire Wire Line
+	2300 3950 2300 4000
+$Comp
+L power:GND #PWR036
+U 1 1 5AF137C0
+P 4400 5450
+F 0 "#PWR036" H 4400 5200 50  0001 C CNN
+F 1 "GND" H 4405 5277 50  0000 C CNN
+F 2 "" H 4400 5450 50  0001 C CNN
+F 3 "" H 4400 5450 50  0001 C CNN
+	1    4400 5450
+	1    0    0    -1
+$EndComp
+$Comp
+L Device:C C10
+U 1 1 5AF137C6
+P 4650 5450
+F 0 "C10" V 4398 5450 50  0000 C CNN
+F 1 "0.1u" V 4489 5450 50  0000 C CNN
+F 2 "Capacitor_SMD:C_0805_2012Metric" H 4688 5300 50  0001 C CNN
+F 3 "~" H 4650 5450 50  0001 C CNN
+	1    4650 5450
+	0    1    1    0
+$EndComp
+Wire Wire Line
+	4400 5450 4500 5450
+Wire Wire Line
+	4800 5450 4900 5450
+Connection ~ 4900 5450
+Wire Wire Line
+	4900 5450 4900 5500
 $EndSCHEMATC

Commit message: LED IND replaced, pcb almost ready
Parts:
- removed U4: CA56-12EWA, Display_7Segment:CA56-12EWA, symbol Display_Character:CA56-12EWA
- added U4: HX3641BH, display-led:HX3641BH, symbol display-led:HX3641BH
Changed lines of the file:
@@
-	1    0    0    -1
-$EndComp
-$Comp
-L Display_Character:CA56-12EWA U4
-U 1 1 5AB7DAD4
-P 5050 4600
-F 0 "U4" H 5100 5167 50  0000 C CNN
-F 1 "CA56-12EWA" H 5100 5076 50  0000 C CNN
-F 2 "Display_7Segment:CA56-12EWA" H 5050 4000 50  0001 C CNN
-F 3 "http://www.kingbrightusa.com/images/catalog/SPEC/CA56-12EWA.pdf" H 4670 4630 50  0001 C CNN
-	1    5050 4600
 	1    0    0    -1
 $EndComp
@@
 Wire Wire Line
 	4900 5450 4900 5500
+$Comp
+L display-led:HX3641BH U4
+U 1 1 5AF54F26
+P 5050 4600
+F 0 "U4" H 5100 5167 50  0000 C CNN
+F 1 "HX3641BH" H 5100 5076 50  0000 C CNN
+F 2 "display-led:HX3641BH" H 5050 4000 50  0001 C CNN
+F 3 "http://www.kingbrightusa.com/images/catalog/SPEC/CA56-12EWA.pdf" H 4670 4630 50  0001 C CNN
+	1    5050 4600
+	1    0    0    -1
+$EndComp
 $EndSCHEMATC

Commit message: added activity indicator for sensor node
Parts:
- added D2: LED, LED_SMD:LED_0805_2012Metric, symbol Device:LED
- added R23: 1k, Resistor_SMD:R_0805_2012Metric, symbol Device:R
Connections:
- wire segments 201 -> 204
Other:
- note added: "Activity indicator for sensor node"
Changed lines of the file:
@@
 	1    0    0    -1
 $EndComp
+Text GLabel 2900 3400 0    50   Output ~ 0
+IND_LATCH
+$Comp
+L Device:LED D2
+U 1 1 5AC005C4
+P 3150 3400
+F 0 "D2" H 3142 3145 50  0000 C CNN
+F 1 "LED" H 3142 3236 50  0000 C CNN
+F 2 "LED_SMD:LED_0805_2012Metric" H 3150 3400 50  0001 C CNN
+F 3 "~" H 3150 3400 50  0001 C CNN
+	1    3150 3400
+	1    0    0    -1
+$EndComp
+$Comp
+L Device:R R23
+U 1 1 5AC00950
+P 3550 3400
+F 0 "R23" V 3757 3400 50  0000 C CNN
+F 1 "1k" V 3666 3400 50  0000 C CNN
+F 2 "Resistor_SMD:R_0805_2012Metric" V 3480 3400 50  0001 C CNN
+F 3 "~" H 3550 3400 50  0001 C CNN
+	1    3550 3400
+	0    1    1    0
+$EndComp
+$Comp
+L power:VCC #PWR038
+U 1 1 5AC00AA8
+P 3800 3400
+F 0 "#PWR038" H 3800 3250 50  0001 C CNN
+F 1 "VCC" H 3817 3573 50  0000 C CNN
+F 2 "" H 3800 3400 50  0001 C CNN
+F 3 "" H 3800 3400 50  0001 C CNN
+	1    3800 3400
+	1    0    0    -1
+$EndComp
+Wire Wire Line
+	2900 3400 3000 3400
+Wire Wire Line
+	3300 3400 3400 3400
+Wire Wire Line
+	3700 3400 3800 3400
+Text Notes 2450 3250 0    50   ~ 0
+Activity indicator for sensor node
 $EndSCHEMATC
