File: pcb/stm8l-lora-sensor.kicad_pcb (KiCad board)
At the start: 2 copper layers, 33 x 57 mm, 50 parts, among them J1 Conn_01x06, J2 Conn_01x02, J3 Conn_01x04, J4 Conn_01x03, J5 Conn_01x02, J6 Conn_01x02, U1 74HC595, U2 STM8L051F3P, U3 74HC595, U4 HX3641BH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

Commit message: pcb: added url
Other:
- board text added: "github.com/dimka-rs/stm8l-lora-sensor"
Changed lines of the file:
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@@
   (general
     (thickness 1.6)
-    (drawings 14)
+    (drawings 15)
     (tracks 620)
     (zones 0)
@@
     (35 F.Paste user hide)
     (36 B.SilkS user)
-    (37 F.SilkS user)
+    (37 F.SilkS user hide)
     (38 B.Mask user hide)
     (39 F.Mask user hide)
@@
     )
   )
+  (gr_text github.com/dimka-rs/stm8l-lora-sensor (at 35 101.5 270) (layer B.SilkS)
+    (effects (font (size 1.5 1.5) (thickness 0.3)) (justify mirror))
+  )
   (gr_arc (start 62 126) (end 62 127) (angle -90) (layer Edge.Cuts) (width 0.15))
